File: Structure_PCB.kicad_pcb (KiCad board)
At the start: 2 copper layers, 180 x 100 mm, 18 parts, among them J5 6620XX236022_662004236022, J6 6620XX236022_662004236022, J7 6620XX236022_662004236022, K2 FINDER-30.22

Commit message: Add files via upload
Routing here
Routing:
- net GND: track 0.00 -> 99.1 mm
- net Net-(D1-K): track 0.00 -> 58.7 mm
- net Net-(J5-Pad3): track 0.00 -> 49.3 mm
- net Net-(J7-Pad1): track 0.00 -> 35.0 mm
- net Net-(J7-Pad3): track 0.00 -> 25.1 mm
- added copper zone on F.Cu, net GND
Changed lines of the file:
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@@
 			(psa4output no)
 			(plot_black_and_white yes)
-			(plotinvisibletext no)
 			(sketchpadsonfab no)
 			(plotpadnumbers no)
@@
 		)
 	)
+	(segment
+		(start 37.82 99.52)
+		(end 49.399 111.099)
+		(width 0.2)
+		(layer "F.Cu")
+		(net 1)
+	)
+	(segment
+		(start 1.5 99.52)
+		(end -1.5 99.52)
+		(width 0.2)
+		(layer "F.Cu")
+		(net 1)
+	)
+	(segment
+		(start -1.5 99.52)
+		(end 37.82 99.52)
+		(width 0.2)
+		(layer "F.Cu")
+		(net 1)
+	)
+	(segment
+		(start -38.265 91.045)
+		(end -17.81 111.5)
+		(width 0.2)
+		(layer "F.Cu")
+		(net 2)
+	)
+	(segment
+		(start -17.81 111.5)
+		(end 49.399 111.5)
+		(width 0.2)
+		(layer "F.Cu")
+		(net 2)
+	)
+	(segment
+		(start -41.265 91.045)
+		(end -38.265 91.045)
+		(width 0.2)
+		(layer "F.Cu")
+		(net 2)
+	)
+	(segment
+		(start -1.5 94.9)
+		(end 1.5 94.9)
+		(width 0.2)
+		(layer "F.Cu")
+		(net 3)
+	)
+	(segment
+		(start -41.265 86.425)
+		(end -9.975 86.425)
+		(width 0.2)
+		(layer "F.Cu")
+		(net 3)
+	)
+	(segment
+		(start -41.265 86.425)
+		(end -38.265 86.425)
+		(width 0.2)
+		(layer "F.Cu")
+		(net 3)
+	)
+	(segment
+		(start -9.975 86.425)
+		(end -1.5 94.9)
+		(width 0.2)
+		(layer "F.Cu")
+		(net 3)
+	)
+	(segment
+		(start 59.48 80)
+		(end 59.48 102.78)
+		(width 0.2)
+		(layer "F.Cu")
+		(net 4)
+	)
+	(segment
+		(start 59.48 77)
+		(end 59.48 80)
+		(width 0.2)
+		(layer "F.Cu")
+		(net 4)
+	)
+	(segment
+		(start 59.48 102.78)
+		(end 58.38 103.88)
+		(width 0.2)
+		(layer "F.Cu")
+		(net 4)
+	)
+	(segment
+		(start 58.38 103.88)
+		(end 66 103.88)
+		(width 0.2)
+		(layer "F.Cu")
+		(net 4)
+	)
+	(segment
+		(start 64.1 91.82)
+		(end 66 93.72)
+		(width 0.2)
+		(layer "F.Cu")
+		(net 5)
+	)
+	(segment
+		(start 64.1 77)
+		(end 64.1 80)
+		(width 0.2)
+		(layer "F.Cu")
+		(net 5)
+	)
+	(segment
+		(start 64.1 80)
+		(end 64.1 91.82)
+		(width 0.2)
+		(layer "F.Cu")
+		(net 5)
+	)
+	(segment
+		(start 66 93.72)
+		(end 58.38 93.72)
+		(width 0.2)
+		(layer "B.Cu")
+		(net 5)
+	)
+	(zone
+		(net 2)
+		(net_name "GND")
+		(layer "F.Cu")
+		(hatch edge 0.5)
+		(connect_pads
+			(clearance 0.5)
+		)
+		(min_thickness 0.25)
+		(filled_areas_thickness no)
+		(fill yes
+			(thermal_gap 0.5)
+			(thermal_bridge_width 0.5)
+		)
+		(polygon
+			(pts
+				(xy 46.3 45.8) (xy 46.3 158.9) (xy 236.8 158.7) (xy 238.3 43.9)
+			)
+		)
+	)
